Commit message: caliberation done

File: linkay_launchfiles/urdf/checker_bot.urdf (robot description, URDF)
Before this commit: robot checker_bot, 4 links, 3 joints
Joints:
- joint laser_1_joint: origin xyz=0.73 0.095 1.43 rpy=0. -0.174533 0. -> xyz=0.73 0.095 1.43 rpy=0. -0.0872665 0.
- joint laser_2_joint: origin xyz=0.73 -0.095 1.43 rpy=0. 0.174533 0. -> xyz=0.73 -0.095 1.43 rpy=0. 0.0872665 0.

Commit message: checker

File: linkay_launchfiles/urdf/checker_bot.urdf (robot description, URDF)
Before this commit: robot checker_bot, 4 links, 3 joints
Joints:
- joint laser_1_joint: origin xyz=0.73 0.095 1.43 rpy=0. -0.0872665 0. -> xyz=0.73 -0.095 1.43 rpy=0. 0.0872665 0.
- joint laser_2_joint: origin xyz=0.73 -0.095 1.43 rpy=0. 0.0872665 0. -> xyz=0.73 0.095 1.43 rpy=0. -0.0872665 0.

Commit message: in blue some checker

File: linkay_launchfiles/urdf/checker_bot.urdf (robot description, URDF)
Before this commit: robot checker_bot, 4 links, 3 joints
Joints:
- joint laser_1_joint: origin xyz=0.73 -0.095 1.43 rpy=0. 0.0872665 0. -> xyz=0.73 -0.095 1.43 rpy=0. 0.0385398 0.
- joint laser_2_joint: origin xyz=0.73 0.095 1.43 rpy=0. -0.0872665 0. -> xyz=0.73 0.095 1.43 rpy=0. -0.0785398 0.

Commit message: blue in the comp

File: linkay_launchfiles/urdf/checker_bot.urdf (robot description, URDF)
Before this commit: robot checker_bot, 4 links, 3 joints
Joints:
- joint laser_1_joint: origin xyz=0.73 -0.095 1.43 rpy=0. 0.0385398 0. -> xyz=0.73 -0.095 1.43 rpy=0. 0.20944 0.
- joint laser_2_joint: origin xyz=0.73 0.095 1.43 rpy=0. -0.0785398 0. -> xyz=0.73 0.095 1.43 rpy=0. -0.20944 0.
